File: dynamixel_3.kicad_sch (KiCad schematic)
At the start: 28 parts, among them J3 Pico5, J4 Dynamixel-3, J5 Dynamixel-3, Q1 MMBT3906, U3 CH343P, U4 SN74LVC1G125DBV, U5 SN74LVC1G126DBVR

Commit message: [update] Positionning v1
Parts:
- D11, D9: value B5819WS -> DNP - B5819WS; now not fitted
- J4, J5: value Dynamixel-3 -> DNP - Dynamixel-3; now not fitted
Changed lines of the file:
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@@
 	(title_block
 		(title "elec_maroilles")
-		(date "2025-11-26")
+		(date "2025-11-28")
 		(rev "A1")
 		(company "Pollen Robotics / Hugging Face")
@@
 	(symbol
 		(lib_id "Device:D_Schottky")
-		(at 317.5 204.47 270)
+		(at 317.5 204.47 90)
+		(mirror x)
 		(unit 1)
 		(exclude_from_sim no)
 		(in_bom yes)
 		(on_board yes)
-		(dnp no)
+		(dnp yes)
 		(property "Reference" "D11"
-			(at 318.516 201.168 90)
+			(at 316.484 201.168 90)
 			(effects
 				(font
@@
 			)
 		)
-		(property "Value" "B5819WS"
-			(at 320.04 205.4224 90)
+		(property "Value" "DNP - B5819WS"
+			(at 314.96 205.4224 90)
 			(effects
 				(font
@@
 		(in_bom yes)
 		(on_board yes)
-		(dnp no)
+		(dnp yes)
 		(property "Reference" "J4"
 			(at 337.82 176.53 0)
@@
 			)
 		)
-		(property "Value" "Dynamixel-3"
+		(property "Value" "DNP - Dynamixel-3"
 			(at 337.82 173.99 0)
 			(effects
@@
 		(in_bom yes)
 		(on_board yes)
-		(dnp no)
+		(dnp yes)
 		(property "Reference" "J5"
 			(at 337.82 191.77 0)
@@
 			)
 		)
-		(property "Value" "Dynamixel-3"
+		(property "Value" "DNP - Dynamixel-3"
 			(at 337.82 189.23 0)
 			(effects
@@
 		(in_bom yes)
 		(on_board yes)
-		(dnp no)
+		(dnp yes)
 		(property "Reference" "D9"
 			(at 315.976 179.324 90)
@@
 			)
 		)
-		(property "Value" "B5819WS"
+		(property "Value" "DNP - B5819WS"
 			(at 314.96 183.8324 90)
 			(effects

Commit message: [update] Release B1!
Parts:
- C3, C5: LCSC Part C302042 -> C1592
- D8: FT Rotation Offset 180 -> (none)
Changed lines of the file:
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@@
 	(title_block
 		(title "elec_maroilles")
-		(date "2025-12-02")
-		(rev "A1")
+		(date "2026-02-02")
+		(rev "B1")
 		(company "Pollen Robotics / Hugging Face")
 	)
@@
 			)
 		)
-		(property "LCSC Part" "C302042"
+		(property "LCSC Part" "C1592"
 			(at 80.01 106.68 0)
 			(effects
@@
 			)
 		)
+		(property "Sim.Device" "PNP"
+			(at 161.29 82.55 0)
+			(effects
+				(font
+					(size 1.27 1.27)
+				)
+				(hide yes)
+			)
+		)
+		(property "Sim.Pins" "1=B 2=E 3=C"
+			(at 161.29 82.55 0)
+			(effects
+				(font
+					(size 1.27 1.27)
+				)
+				(hide yes)
+			)
+		)
 		(pin "2"
 		)
@@
 			)
 		)
-		(property "LCSC Part" "C302042"
+		(property "LCSC Part" "C1592"
 			(at 74.93 106.68 0)
 			(effects
@@
 			)
 		)
-		(property "FT Rotation Offset" "180"
+		(property "FT Rotation Offset" ""
 			(at 288.29 184.15 90)
 			(effects
